Commit message: working model

File: agv_gazebo_sim/urdf/m2wr.xacro (robot description, xacro)
@@ -1,7 +1,7 @@
 <?xml version="1.0" ?>
 <robot name="m2wr" xmlns:xacro="http://www.ros.org/wiki/xacro">
-  <xacro:include filename="$(find m2wr_description)/urdf/materials.xacro" />
-  <xacro:include filename="$(find m2wr_description)/urdf/m2wr.gazebo" />
-  <xacro:include filename="$(find m2wr_description)/urdf/macros.xacro" />
+  <xacro:include filename="$(find agv_gazebo_sim)/urdf/materials.xacro" />
+  <xacro:include filename="$(find agv_gazebo_sim)/urdf/m2wr.gazebo" />
+  <xacro:include filename="$(find agv_gazebo_sim)/urdf/macros.xacro" />
   <link name="base_link">
     <!-- pose and inertial -->
@@ -21,5 +21,5 @@
       <origin rpy="0 0 0" xyz="0 0 0.01"/>
       <geometry>
-        <mesh filename="file://$(find m2wr_description)/models/v1/meshes/cart.dae"  scale="1 1 1"/>
+        <mesh filename="file://$(find agv_gazebo_sim)/models/v1/meshes/cart.dae"  scale="1 1 1"/>
       </geometry>
       <material name="blue"/>
